File: GlitchPixel404.kicad_sch (KiCad schematic)
At the start: 76 parts, among them J1 Barrel_Jack_Switch, J2 TYPE-C-31-M-12, J3 VOLTLINK, J4 Conn_01x03, J5 Output, Q1 AONR21357-ES, Q2 MMBT3904, SW1 Reset, SW2 Boot, SW3 SW_SP3T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

Commit message: Update silkscreen
Parts:
- J1: now fitted; now in the parts list
Other:
- moved on the sheet: TPr2
Changed lines of the file:
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@@
 	(wire
 		(pts
+			(xy 50.8 44.45) (xy 49.53 44.45)
+		)
+		(stroke
+			(width 0)
+			(type default)
+		)
+	)
+	(wire
+		(pts
 			(xy 100.33 119.38) (xy 92.71 119.38)
 		)
@@
 		)
 		(instances
-			(project ""
+			(project "GlitchPixel404"
 				(path "/3cfb80c9-371d-4841-9148-eae536d7cb55"
 					(reference "C1")
@@
 		)
 		(instances
-			(project ""
+			(project "GlitchPixel404"
 				(path "/3cfb80c9-371d-4841-9148-eae536d7cb55"
 					(reference "U3")
@@
 		)
 		(instances
-			(project ""
+			(project "GlitchPixel404"
 				(path "/3cfb80c9-371d-4841-9148-eae536d7cb55"
 					(reference "MK1")
@@
 	(symbol
 		(lib_id "Connector:TestPoint_Small")
-		(at 49.53 44.45 0)
+		(at 50.8 44.45 0)
 		(unit 1)
 		(exclude_from_sim no)
@@
 		(fields_autoplaced yes)
 		(property "Reference" "TPr2"
-			(at 50.8 43.1799 0)
+			(at 52.07 43.1799 0)
 			(effects
 				(font
@@
 		)
 		(property "Value" "Vbus"
-			(at 50.8 45.7199 0)
+			(at 52.07 45.7199 0)
 			(effects
 				(font
@@
 		)
 		(property "Footprint" "TestPoint:TestPoint_Pad_D1.0mm"
-			(at 54.61 44.45 0)
+			(at 55.88 44.45 0)
 			(effects
 				(font
@@
 		)
 		(property "Datasheet" "~"
-			(at 54.61 44.45 0)
+			(at 55.88 44.45 0)
 			(effects
 				(font
@@
 		)
 		(property "Description" "test point"
-			(at 49.53 44.45 0)
+			(at 50.8 44.45 0)
 			(effects
 				(font
@@
 		)
 		(instances
-			(project ""
+			(project "GlitchPixel404"
 				(path "/3cfb80c9-371d-4841-9148-eae536d7cb55"
 					(reference "#PWR02")
@@
 		)
 		(instances
-			(project ""
+			(project "GlitchPixel404"
 				(path "/3cfb80c9-371d-4841-9148-eae536d7cb55"
 					(reference "D4")
@@
 		)
 		(instances
-			(project ""
+			(project "GlitchPixel404"
 				(path "/3cfb80c9-371d-4841-9148-eae536d7cb55"
 					(reference "R5")
@@
 		)
 		(instances
-			(project ""
+			(project "GlitchPixel404"
 				(path "/3cfb80c9-371d-4841-9148-eae536d7cb55"
 					(reference "U4")
@@
 		)
 		(instances
-			(project ""
+			(project "GlitchPixel404"
 				(path "/3cfb80c9-371d-4841-9148-eae536d7cb55"
 					(reference "C13")
@@
 		)
 		(instances
-			(project ""
+			(project "GlitchPixel404"
 				(path "/3cfb80c9-371d-4841-9148-eae536d7cb55"
 					(reference "J2")
@@
 		)
 		(instances
-			(project ""
+			(project "GlitchPixel404"
 				(path "/3cfb80c9-371d-4841-9148-eae536d7cb55"
 					(reference "D5")
@@
 		)
 		(instances
-			(project ""
+			(project "GlitchPixel404"
 				(path "/3cfb80c9-371d-4841-9148-eae536d7cb55"
 					(reference "TPr3")
@@
 		)
 		(instances
-			(project ""
+			(project "GlitchPixel404"
 				(path "/3cfb80c9-371d-4841-9148-eae536d7cb55"
 					(reference "Q2")
@@
 		)
 		(instances
-			(project ""
+			(project "GlitchPixel404"
 				(path "/3cfb80c9-371d-4841-9148-eae536d7cb55"
 					(reference "SW3")
@@
 		)
 		(instances
-			(project ""
+			(project "GlitchPixel404"
 				(path "/3cfb80c9-371d-4841-9148-eae536d7cb55"
 					(reference "U6")
@@
 		)
 		(instances
-			(project ""
+			(project "GlitchPixel404"
 				(path "/3cfb80c9-371d-4841-9148-eae536d7cb55"
 					(reference "C5")
@@
 		)
 		(instances
-			(project ""
+			(project "GlitchPixel404"
 				(path "/3cfb80c9-371d-4841-9148-eae536d7cb55"
 					(reference "#PWR027")
@@
 		)
 		(instances
-			(project ""
+			(project "GlitchPixel404"
 				(path "/3cfb80c9-371d-4841-9148-eae536d7cb55"
 					(reference "U5")
@@
 		(unit 1)
 		(exclude_from_sim no)
-		(in_bom no)
+		(in_bom yes)
 		(on_board yes)
-		(dnp yes)
+		(dnp no)
 		(fields_autoplaced yes)
 		(property "Reference" "J1"
@@
 		)
 		(instances
-			(project ""
+			(project "GlitchPixel404"
 				(path "/3cfb80c9-371d-4841-9148-eae536d7cb55"
 					(reference "J1")
@@
 		)
 		(instances
-			(project ""
+			(project "GlitchPixel404"
 				(path "/3cfb80c9-371d-4841-9148-eae536d7cb55"
 					(reference "J5")
@@
 		)
 		(instances
-			(project ""
+			(project "GlitchPixel404"
 				(path "/3cfb80c9-371d-4841-9148-eae536d7cb55"
 					(reference "L1")
@@
 		)
 		(instances
-			(project ""
+			(project "GlitchPixel404"
 				(path "/3cfb80c9-371d-4841-9148-eae536d7cb55"
 					(reference "#PWR021")
@@
 		)
 		(instances
-			(project ""
+			(project "GlitchPixel404"
 				(path "/3cfb80c9-371d-4841-9148-eae536d7cb55"
 					(reference "J4")
@@
 		)
 		(instances
-			(project ""
+			(project "GlitchPixel404"
 				(path "/3cfb80c9-371d-4841-9148-eae536d7cb55"
 					(reference "Ue1")
@@
 		)
 		(instances
-			(project ""
+			(project "GlitchPixel404"
 				(path "/3cfb80c9-371d-4841-9148-eae536d7cb55"
 					(reference "Q1")
@@
 		)
 		(instances
-			(project ""
+			(project "GlitchPixel404"
 				(path "/3cfb80c9-371d-4841-9148-eae536d7cb55"
 					(reference "D1")
@@
 		)
 		(instances
-			(project ""
+			(project "GlitchPixel404"
 				(path "/3cfb80c9-371d-4841-9148-eae536d7cb55"
 					(reference "F1")
@@
 		)
 		(instances
-			(project ""
+			(project "GlitchPixel404"
 				(path "/3cfb80c9-371d-4841-9148-eae536d7cb55"
 					(reference "U1")
@@
 		)
 		(instances
-			(project ""
+			(project "GlitchPixel404"
 				(path "/3cfb80c9-371d-4841-9148-eae536d7cb55"
 					(reference "D2")
@@
 		)
 		(instances
-			(project ""
+			(project "GlitchPixel404"
 				(path "/3cfb80c9-371d-4841-9148-eae536d7cb55"
 					(reference "H1")
